File: hardware/power.kicad_sch (KiCad schematic)
At the start: 8 parts, among them U3 LD1086DT50TR, U4 AMS1117-3.3

Commit message: power silindi ve sim800l çizildi
Parts:
- removed C10, C14: 22u, symbol Device:C
- removed C17, C18: 10uF, symbol Device:C_Polarized
- removed LD1: RED, symbol Device:D_Laser_1C2A
- removed R13: 1k5, symbol Device:R
- removed U3: LD1086DT50TR, Package_TO_SOT_SMD:TO-252-2, symbol Regulator_Linear:LD1086DT50TR
- removed U4: AMS1117-3.3, Package_TO_SOT_SMD:SOT-223-3_TabPin2, symbol Regulator_Linear:AMS1117

Commit message: Power ve ADC sematikleri çizildi
Parts:
- added C10, C14: 22u, symbol Device:C
- added C17, C18: 10uF, symbol Device:C_Polarized
- added LD1: RED, symbol Device:D_Laser_1C2A
- added R13: 1k5, symbol Device:R
- added U3: LD1086DT50TR, Package_TO_SOT_SMD:TO-252-2, symbol Regulator_Linear:LD1086DT50TR
- added U4: AMS1117-3.3, Package_TO_SOT_SMD:SOT-223-3_TabPin2, symbol Regulator_Linear:AMS1117
Connections:
- new net: LD1.1 (K), R13.1
- new net +3.3V: C14.1, LD1.2 (A), U4.2 (VO)
- new net +5V: C10.1, C17.1, U3.2 (OUT), U4.3 (VI)
- new net GND: C10.2, C14.2, C17.2, C18.2, R13.2, U3.1 (ADJ/GND), U4.1 (ADJ)
- new net INPUT: 12V: C18.1, U3.3 (IN)
