File: hardware/lcd.kicad_sch (KiCad schematic)
At the start: 0 parts

Commit message: LCD module completed
Parts:
- added Brd1: SSD1306, 2023Staj:SSD1306_0.96_Oled, symbol 2023Staj:SSD1306
Connections:
- new net +5V: Brd1.2 (VCC)
- new net GND: Brd1.1 (GND)
- new net SCL: Brd1.3 (SCL)
- new net SDA: Brd1.4 (SDA)
Changed lines of the file:
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@@
 (kicad_sch (version 20230121) (generator eeschema)
   (paper "A4")
+  (wire (pts (xy 144.78 80.01) (xy 154.94 80.01))
+    (stroke (width 0) (type default))
+  )
+  (wire (pts (xy 143.51 82.55) (xy 154.94 82.55))
+    (stroke (width 0) (type default))
+  )
+  (wire (pts (xy 154.94 77.47) (xy 148.59 77.47))
+    (stroke (width 0) (type default))
+  )
+  (wire (pts (xy 144.78 69.85) (xy 144.78 80.01))
+    (stroke (width 0) (type default))
+  )
+  (wire (pts (xy 148.59 77.47) (xy 148.59 93.98))
+    (stroke (width 0) (type default))
+  )
+  (wire (pts (xy 143.51 85.09) (xy 154.94 85.09))
+    (stroke (width 0) (type default))
+  )
+  (hierarchical_label "SDA" (shape bidirectional) (at 143.51 85.09 180) (fields_autoplaced)
+    (effects (font (size 1.27 1.27)) (justify right))
+  )
+  (hierarchical_label "SCL" (shape input) (at 143.51 82.55 180) (fields_autoplaced)
+    (effects (font (size 1.27 1.27)) (justify right))
+  )
+  (symbol (lib_id "2023Staj:SSD1306") (at 163.83 81.28 90) (mirror x) (unit 1)
+    (in_bom yes) (on_board yes) (dnp no)
+    (property "Reference" "Brd1" (at 157.48 73.66 90)
+      (effects (font (size 1.27 1.27)) (justify right))
+    )
+    (property "Value" "SSD1306" (at 162.56 88.9 90)
+      (effects (font (size 1.27 1.27)) (justify right))
+    )
+    (property "Footprint" "2023Staj:SSD1306_0.96_Oled" (at 157.48 81.28 0)
+      (effects (font (size 1.27 1.27)) hide)
+    )
+    (property "Datasheet" "" (at 157.48 81.28 0)
+      (effects (font (size 1.27 1.27)) hide)
+    )
+    (pin "1")
+    (pin "2")
+    (pin "3")
+    (pin "4")
+    (instances
+      (project "2023-staj-projesi"
+        (path "/069db7ad-35cd-4aa8-8111-e026f632a4df/9df18327-ad01-4780-8291-2b0f280e8588"
+          (reference "Brd1") (unit 1)
+        )
+      )
+    )
+  )
+  (symbol (lib_id "power:+5V") (at 144.78 69.85 0) (unit 1)
+    (in_bom yes) (on_board yes) (dnp no) (fields_autoplaced)
+    (property "Reference" "#PWR025" (at 144.78 73.66 0)
+      (effects (font (size 1.27 1.27)) hide)
+    )
+    (property "Value" "+5V" (at 144.78 64.77 0)
+      (effects (font (size 1.27 1.27)))
+    )
+    (property "Footprint" "" (at 144.78 69.85 0)
+      (effects (font (size 1.27 1.27)) hide)
+    )
+    (property "Datasheet" "" (at 144.78 69.85 0)
+      (effects (font (size 1.27 1.27)) hide)
+    )
+    (pin "1")
+    (instances
+      (project "2023-staj-projesi"
+        (path "/069db7ad-35cd-4aa8-8111-e026f632a4df/9df18327-ad01-4780-8291-2b0f280e8588"
+          (reference "#PWR025") (unit 1)
+        )
+      )
+    )
+  )
+  (symbol (lib_id "power:GND") (at 148.59 93.98 0) (unit 1)
+    (in_bom yes) (on_board yes) (dnp no) (fields_autoplaced)
+    (property "Reference" "#PWR024" (at 148.59 100.33 0)
+      (effects (font (size 1.27 1.27)) hide)
+    )
+    (property "Value" "GND" (at 148.59 99.06 0)
+      (effects (font (size 1.27 1.27)))
+    )
+    (property "Footprint" "" (at 148.59 93.98 0)
+      (effects (font (size 1.27 1.27)) hide)
+    )
+    (property "Datasheet" "" (at 148.59 93.98 0)
+      (effects (font (size 1.27 1.27)) hide)
+    )
+    (pin "1")
+    (instances
+      (project "2023-staj-projesi"
+        (path "/069db7ad-35cd-4aa8-8111-e026f632a4df/9df18327-ad01-4780-8291-2b0f280e8588"
+          (reference "#PWR024") (unit 1)
+        )
+      )
+    )
+  )
 )
